File: Hardware/SHTC3 Breakout.sch (EAGLE design)
At the start: 22 parts, among them J2 QWIIC_RIGHT_ANGLE, J3 PTH, J4 QWIIC_RIGHT_ANGLE, U1 SHTC3

Commit message: pre review commit
Other:
- moved on the sheet: C1
Changed lines of the file:
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@@
 <attribute name="VALUE" x="142.24" y="152.654" size="1.778" layer="96" font="vector" align="bottom-center"/>
 </instance>
-<instance part="C1" gate="G$1" x="63.5" y="124.46" smashed="yes">
-<attribute name="NAME" x="65.024" y="127.381" size="1.778" layer="95" font="vector"/>
-<attribute name="VALUE" x="65.024" y="122.301" size="1.778" layer="96" font="vector"/>
+<instance part="C1" gate="G$1" x="68.58" y="124.46" smashed="yes">
+<attribute name="NAME" x="70.104" y="127.381" size="1.778" layer="95" font="vector"/>
+<attribute name="VALUE" x="70.104" y="122.301" size="1.778" layer="96" font="vector"/>
 </instance>
-<instance part="SUPPLY3" gate="G$1" x="63.5" y="132.08" smashed="yes">
-<attribute name="VALUE" x="63.5" y="134.874" size="1.778" layer="96" font="vector" align="bottom-center"/>
+<instance part="SUPPLY3" gate="G$1" x="68.58" y="132.08" smashed="yes">
+<attribute name="VALUE" x="68.58" y="134.874" size="1.778" layer="96" font="vector" align="bottom-center"/>
 </instance>
-<instance part="GND2" gate="1" x="63.5" y="116.84" smashed="yes">
-<attribute name="VALUE" x="60.96" y="114.3" size="1.778" layer="96" font="vector"/>
+<instance part="GND2" gate="1" x="68.58" y="116.84" smashed="yes">
+<attribute name="VALUE" x="66.04" y="114.3" size="1.778" layer="96" font="vector"/>
 </instance>
 <instance part="LOGO2" gate="G$1" x="190.5" y="40.64" smashed="yes"/>
@@
 <pinref part="C1" gate="G$1" pin="1"/>
 <pinref part="SUPPLY3" gate="G$1" pin="3.3V"/>
-<wire x1="63.5" y1="129.54" x2="63.5" y2="132.08" width="0.1524" layer="91"/>
+<wire x1="68.58" y1="129.54" x2="68.58" y2="132.08" width="0.1524" layer="91"/>
 </segment>
 <segment>
@@
 <pinref part="GND2" gate="1" pin="GND"/>
 <pinref part="C1" gate="G$1" pin="2"/>
-<wire x1="63.5" y1="119.38" x2="63.5" y2="121.92" width="0.1524" layer="91"/>
+<wire x1="68.58" y1="119.38" x2="68.58" y2="121.92" width="0.1524" layer="91"/>
 </segment>
 </net>

Commit message: post review/checklist changes, ready for QC double check
Parts:
- removed J3: PTH, SparkX:I2C_STANDARD_NO_SILK
- removed PWR: JUMPER-SMT_2_NC_TRACE_NO-SILK, SparkFun-Jumpers:JUMPER-SMT_2_NC_TRACE_NO-SILK
- added J1: (no value), SparkFun-Connectors:CONN_041X04_NO_SILK
- added JP7, JP8: STAND-OFF, SparkFun:STAND-OFF
- added PWRLED: JUMPER-SMT_2_NC_TRACE_SILK, SparkFun-Jumpers:JUMPER-SMT_2_NC_TRACE_SILK
- U1: device SHTC3:SHTC3 -> SparkFun-Sensors:SHTC3
Connections:
- net 3.3V: now also J1.2, PWRLED.2; no longer J3.VCC, PWR.2
- net GND: now also J1.1; no longer J3.GND
- net N$4: now also PWRLED.1; no longer PWR.1
- net SCL: now also J1.4; no longer J3.SCL
- net SDA: now also J1.3; no longer J3.SDA
Other:
- note added: "VIN: 1.62-3.6V"
Changed lines of the file:
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@@
 <part name="GND6" library="SparkFun" deviceset="GND" device=""/>
 <part name="SUPPLY7" library="SparkFun-PowerSymbols" deviceset="3.3V" device=""/>
-<part name="J3" library="SparkX" deviceset="I2C_STANDARD" device="_NO_SILK" value="PTH"/>
 <part name="GND7" library="SparkFun" deviceset="GND" device=""/>
 <part name="FRAME1" library="SparkFun-Aesthetics" deviceset="FRAME-LETTER" device=""/>
@@
 <part name="D1" library="SparkFun-LED" deviceset="LED-RED" device="0603" value="RED"/>
 <part name="GND3" library="SparkFun" deviceset="GND" device=""/>
-<part name="U1" library="SHTC3" deviceset="SHTC3" device=""/>
+<part name="U1" library="SparkFun-Sensors" deviceset="SHTC3" device="" value="SHTC3"/>
 <part name="R1" library="SparkFun-Resistors" deviceset="2.2KOHM" device="-0603-1/10W-1%" value="2.2k"/>
 <part name="R2" library="SparkFun-Resistors" deviceset="2.2KOHM" device="-0603-1/10W-1%" value="2.2k"/>
@@
 <part name="LOGO2" library="SparkFun-Aesthetics" deviceset="SFE_LOGO_NAME_FLAME" device=".1_INCH"/>
 <part name="LOGO3" library="SparkFun-Aesthetics" deviceset="SFE_LOGO_NAME_FLAME" device=".1_INCH"/>
-<part name="PWR" library="SparkFun-Jumpers" deviceset="JUMPER-SMT_2_NC_TRACE" device="_NO-SILK" package3d_urn="urn:adsk.eagle:package:39286/1" value="JUMPER-SMT_2_NC_TRACE_NO-SILK"/>
+<part name="PWRLED" library="SparkFun-Jumpers" deviceset="JUMPER-SMT_2_NC_TRACE" device="_SILK" package3d_urn="urn:adsk.eagle:package:39281/1" value="JUMPER-SMT_2_NC_TRACE_SILK"/>
 <part name="LOGO4" library="SparkFun-Aesthetics" deviceset="REVISION" device=""/>
+<part name="JP7" library="SparkFun" deviceset="STAND-OFF" device=""/>
+<part name="JP8" library="SparkFun" deviceset="STAND-OFF" device=""/>
+<part name="J1" library="SparkFun-Connectors" deviceset="CONN_04" device="1X04_NO_SILK"/>
 </parts>
 <sheets>
@@
 the power LED</text>
 <text x="169.418" y="7.874" size="2.54" layer="94" font="vector">Andy England</text>
+<text x="105.918" y="163.068" size="1.778" layer="97" font="vector">VIN: 1.62-3.6V</text>
 </plain>
 <instances>
@@
 <attribute name="VALUE" x="76.2" y="56.134" size="1.778" layer="96" font="vector" align="bottom-center"/>
 </instance>
-<instance part="J3" gate="G$1" x="86.36" y="45.72" smashed="yes" rot="MR0">
-<attribute name="VALUE" x="91.44" y="40.386" size="1.778" layer="96" font="vector" rot="MR0" align="top-left"/>
-<attribute name="NAME" x="91.44" y="53.594" size="1.778" layer="95" font="vector" rot="MR0"/>
-</instance>
 <instance part="GND7" gate="1" x="76.2" y="38.1" smashed="yes">
 <attribute name="VALUE" x="73.66" y="35.56" size="1.778" layer="96" font="vector"/>
@@
 <instance part="LOGO2" gate="G$1" x="190.5" y="40.64" smashed="yes"/>
 <instance part="LOGO3" gate="G$1" x="190.5" y="40.64" smashed="yes"/>
-<instance part="PWR" gate="G$1" x="33.02" y="139.7" smashed="yes" rot="R90">
+<instance part="PWRLED" gate="G$1" x="33.02" y="139.7" smashed="yes" rot="R90">
 <attribute name="NAME" x="35.56" y="139.7" size="1.778" layer="95" font="vector"/>
 </instance>
 <instance part="LOGO4" gate="G$1" x="148.844" y="7.874" smashed="yes"/>
+<instance part="JP7" gate="G$1" x="243.84" y="30.48" smashed="yes"/>
+<instance part="JP8" gate="G$1" x="243.84" y="27.94" smashed="yes"/>
+<instance part="J1" gate="J1" x="83.82" y="45.72" smashed="yes" rot="MR0">
+<attribute name="VALUE" x="88.9" y="38.354" size="1.778" layer="96" font="vector" rot="MR0"/>
+<attribute name="NAME" x="88.9" y="53.848" size="1.778" layer="95" font="vector" rot="MR0"/>
+</instance>
 </instances>
 <busses>
@@
 </segment>
 <segment>
-<pinref part="J3" gate="G$1" pin="VCC"/>
 <wire x1="78.74" y1="45.72" x2="76.2" y2="45.72" width="0.1524" layer="91"/>
 <wire x1="76.2" y1="45.72" x2="76.2" y2="53.34" width="0.1524" layer="91"/>
 <pinref part="SUPPLY7" gate="G$1" pin="3.3V"/>
+<pinref part="J1" gate="J1" pin="2"/>
 </segment>
 <segment>
@@
 <segment>
 <pinref part="SUPPLY10" gate="G$1" pin="3.3V"/>
-<pinref part="PWR" gate="G$1" pin="2"/>
+<pinref part="PWRLED" gate="G$1" pin="2"/>
 <wire x1="33.02" y1="147.32" x2="33.02" y2="144.78" width="0.1524" layer="91"/>
 </segment>
@@
 </segment>
 <segment>
-<pinref part="J3" gate="G$1" pin="GND"/>
 <wire x1="78.74" y1="43.18" x2="76.2" y2="43.18" width="0.1524" layer="91"/>
 <wire x1="76.2" y1="43.18" x2="76.2" y2="40.64" width="0.1524" layer="91"/>
 <pinref part="GND7" gate="1" pin="GND"/>
+<pinref part="J1" gate="J1" pin="1"/>
 </segment>
 <segment>
@@
 </segment>
 <segment>
-<pinref part="J3" gate="G$1" pin="SCL"/>
 <wire x1="78.74" y1="50.8" x2="73.66" y2="50.8" width="0.1524" layer="91"/>
 <label x="73.66" y="50.8" size="1.27" layer="95" font="vector" rot="R180" xref="yes"/>
+<pinref part="J1" gate="J1" pin="4"/>
 </segment>
 <segment>
@@
 </segment>
 <segment>
-<pinref part="J3" gate="G$1" pin="SDA"/>
 <wire x1="78.74" y1="48.26" x2="73.66" y2="48.26" width="0.1524" layer="91"/>
 <label x="73.66" y="48.26" size="1.27" layer="95" font="vector" rot="R180" xref="yes"/>
+<pinref part="J1" gate="J1" pin="3"/>
 </segment>
 <segment>
@@
 <net name="N$4" class="0">
 <segment>
-<pinref part="PWR" gate="G$1" pin="1"/>
+<pinref part="PWRLED" gate="G$1" pin="1"/>
 <pinref part="R3" gate="G$1" pin="2"/>
 <wire x1="33.02" y1="134.62" x2="33.02" y2="132.08" width="0.1524" layer="91"/>
